File: sensor/sensor.kicad_sch (KiCad schematic)
At the start: 6 parts, among them U1 LM358

Commit message: Mostly finallized PCB
Parts:
- added R4, R5: 1k, symbol Device:R
- added unit 3 of U1
- added unit 2 of U1
Connections:
- net +5V: now also R4.1, U1.8 (V+)
- net GND: now also R5.2, U1.4 (V-)
- new net: R4.2, R5.1, U1.5 (+)
- new net: U1.6 (-), U1.7
Changed lines of the file:
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@@
   (junction (at 48.26 46.99) (diameter 0) (color 0 0 0 0)
   )
+  (junction (at 63.5 73.66) (diameter 0) (color 0 0 0 0)
+  )
   (junction (at 25.4 34.29) (diameter 0) (color 0 0 0 0)
   )
@@
     (stroke (width 0) (type default))
   )
+  (wire (pts (xy 63.5 71.12) (xy 63.5 73.66))
+    (stroke (width 0) (type default))
+  )
+  (wire (pts (xy 73.66 78.74) (xy 72.39 78.74))
+    (stroke (width 0) (type default))
+  )
+  (wire (pts (xy 91.44 83.82) (xy 91.44 76.2))
+    (stroke (width 0) (type default))
+  )
+  (wire (pts (xy 91.44 76.2) (xy 88.9 76.2))
+    (stroke (width 0) (type default))
+  )
   (wire (pts (xy 69.85 30.48) (xy 69.85 40.64))
     (stroke (width 0) (type default))
   )
+  (wire (pts (xy 72.39 78.74) (xy 72.39 83.82))
+    (stroke (width 0) (type default))
+  )
+  (wire (pts (xy 63.5 73.66) (xy 63.5 76.2))
+    (stroke (width 0) (type default))
+  )
   (wire (pts (xy 48.26 46.99) (xy 69.85 46.99))
     (stroke (width 0) (type default))
@@
   )
   (wire (pts (xy 25.4 34.29) (xy 55.88 34.29))
+    (stroke (width 0) (type default))
+  )
+  (wire (pts (xy 63.5 73.66) (xy 73.66 73.66))
+    (stroke (width 0) (type default))
+  )
+  (wire (pts (xy 72.39 83.82) (xy 91.44 83.82))
     (stroke (width 0) (type default))
   )
@@
         (path "/2513f109-8989-495f-b5d5-45fde763de5f"
           (reference "LD1") (unit 1)
+        )
+      )
+    )
+  )
+  (symbol (lib_id "Device:R") (at 63.5 80.01 0) (unit 1)
+    (in_bom yes) (on_board yes) (dnp no) (fields_autoplaced)
+    (property "Reference" "R5" (at 65.278 78.7979 0)
+      (effects (font (size 1.27 1.27)) (justify left))
+    )
+    (property "Value" "1k" (at 65.278 81.2221 0)
+      (effects (font (size 1.27 1.27)) (justify left))
+    )
+    (property "Footprint" "" (at 61.722 80.01 90)
+      (effects (font (size 1.27 1.27)) hide)
+    )
+    (property "Datasheet" "~" (at 63.5 80.01 0)
+      (effects (font (size 1.27 1.27)) hide)
+    )
+    (pin "1")
+    (pin "2")
+    (instances
+      (project "sensor"
+        (path "/2513f109-8989-495f-b5d5-45fde763de5f"
+          (reference "R5") (unit 1)
         )
       )
@@
     )
   )
+  (symbol (lib_id "power:GND") (at 63.5 83.82 0) (unit 1)
+    (in_bom yes) (on_board yes) (dnp no) (fields_autoplaced)
+    (property "Reference" "#PWR09" (at 63.5 90.17 0)
+      (effects (font (size 1.27 1.27)) hide)
+    )
+    (property "Value" "GND" (at 63.5 87.9531 0)
+      (effects (font (size 1.27 1.27)))
+    )
+    (property "Footprint" "" (at 63.5 83.82 0)
+      (effects (font (size 1.27 1.27)) hide)
+    )
+    (property "Datasheet" "" (at 63.5 83.82 0)
+      (effects (font (size 1.27 1.27)) hide)
+    )
+    (pin "1")
+    (instances
+      (project "sensor"
+        (path "/2513f109-8989-495f-b5d5-45fde763de5f"
+          (reference "#PWR09") (unit 1)
+        )
+      )
+    )
+  )
   (symbol (lib_id "power:GND") (at 48.26 39.37 180) (unit 1)
     (in_bom yes) (on_board yes) (dnp no) (fields_autoplaced)
@@
       (effects (font (size 1.27 1.27)) hide)
     )
-    (property "Value" "GND" (at 48.26 35.56 0)
-      (effects (font (size 1.27 1.27)))
+    (property "Value" "GND" (at 50.165 38.1 0)
+      (effects (font (size 1.27 1.27)) (justify right))
     )
     (property "Footprint" "" (at 48.26 39.37 0)
@@
     )
   )
+  (symbol (lib_id "Amplifier_Operational:LM358") (at 27.94 85.09 0) (unit 3)
+    (in_bom yes) (on_board yes) (dnp no) (fields_autoplaced)
+    (property "Reference" "U1" (at 26.035 83.8779 0)
+      (effects (font (size 1.27 1.27)) (justify left))
+    )
+    (property "Value" "LM358" (at 26.035 86.3021 0)
+      (effects (font (size 1.27 1.27)) (justify left))
+    )
+    (property "Footprint" "" (at 27.94 85.09 0)
+      (effects (font (size 1.27 1.27)) hide)
+    )
+    (property "Datasheet" "http://www.ti.com/lit/ds/symlink/lm2904-n.pdf" (at 27.94 85.09 0)
+      (effects (font (size 1.27 1.27)) hide)
+    )
+    (pin "1")
+    (pin "2")
+    (pin "3")
+    (pin "5")
+    (pin "6")
+    (pin "7")
+    (pin "4")
+    (pin "8")
+    (instances
+      (project "sensor"
+        (path "/2513f109-8989-495f-b5d5-45fde763de5f"
+          (reference "U1") (unit 3)
+        )
+      )
+    )
+  )
+  (symbol (lib_id "power:+5V") (at 25.4 77.47 0) (unit 1)
+    (in_bom yes) (on_board yes) (dnp no) (fields_autoplaced)
+    (property "Reference" "#PWR06" (at 25.4 81.28 0)
+      (effects (font (size 1.27 1.27)) hide)
+    )
+    (property "Value" "+5V" (at 25.4 73.3369 0)
+      (effects (font (size 1.27 1.27)))
+    )
+    (property "Footprint" "" (at 25.4 77.47 0)
+      (effects (font (size 1.27 1.27)) hide)
+    )
+    (property "Datasheet" "" (at 25.4 77.47 0)
+      (effects (font (size 1.27 1.27)) hide)
+    )
+    (pin "1")
+    (instances
+      (project "sensor"
+        (path "/2513f109-8989-495f-b5d5-45fde763de5f"
+          (reference "#PWR06") (unit 1)
+        )
+      )
+    )
+  )
+  (symbol (lib_id "power:GND") (at 25.4 92.71 0) (unit 1)
+    (in_bom yes) (on_board yes) (dnp no) (fields_autoplaced)
+    (property "Reference" "#PWR07" (at 25.4 99.06 0)
+      (effects (font (size 1.27 1.27)) hide)
+    )
+    (property "Value" "GND" (at 25.4 96.8431 0)
+      (effects (font (size 1.27 1.27)))
+    )
+    (property "Footprint" "" (at 25.4 92.71 0)
+      (effects (font (size 1.27 1.27)) hide)
+    )
+    (property "Datasheet" "" (at 25.4 92.71 0)
+      (effects (font (size 1.27 1.27)) hide)
+    )
+    (pin "1")
+    (instances
+      (project "sensor"
+        (path "/2513f109-8989-495f-b5d5-45fde763de5f"
+          (reference "#PWR07") (unit 1)
+        )
+      )
+    )
+  )
   (symbol (lib_id "power:+5V") (at 25.4 62.23 180) (unit 1)
     (in_bom yes) (on_board yes) (dnp no) (fields_autoplaced)
@@
         )
       )
+    )
+  )
+  (symbol (lib_id "Device:R") (at 63.5 67.31 0) (unit 1)
+    (in_bom yes) (on_board yes) (dnp no) (fields_autoplaced)
+    (property "Reference" "R4" (at 65.278 66.0979 0)
+      (effects (font (size 1.27 1.27)) (justify left))
+    )
+    (property "Value" "1k" (at 65.278 68.5221 0)
+      (effects (font (size 1.27 1.27)) (justify left))
+    )
+    (property "Footprint" "" (at 61.722 67.31 90)
+      (effects (font (size 1.27 1.27)) hide)
+    )
+    (property "Datasheet" "~" (at 63.5 67.31 0)
+      (effects (font (size 1.27 1.27)) hide)
+    )
+    (pin "1")
+    (pin "2")
+    (instances
+      (project "sensor"
+        (path "/2513f109-8989-495f-b5d5-45fde763de5f"
+          (reference "R4") (unit 1)
+        )
+      )
+    )
+  )
+  (symbol (lib_id "power:+5V") (at 63.5 63.5 0) (unit 1)
+    (in_bom yes) (on_board yes) (dnp no) (fields_autoplaced)
+    (property "Reference" "#PWR08" (at 63.5 67.31 0)
+      (effects (font (size 1.27 1.27)) hide)
+    )
+    (property "Value" "+5V" (at 63.5 59.3669 0)
+      (effects (font (size 1.27 1.27)))
+    )
+    (property "Footprint" "" (at 63.5 63.5 0)
+      (effects (font (size 1.27 1.27)) hide)
+    )
+    (property "Datasheet" "" (at 63.5 63.5 0)
+      (effects (font (size 1.27 1.27)) hide)
+    )
+    (pin "1")
+    (instances
+      (project "sensor"
+        (path "/2513f109-8989-495f-b5d5-45fde763de5f"
+          (reference "#PWR08") (unit 1)
+        )
+      )
+    )
+  )
+  (symbol (lib_id "Amplifier_Operational:LM358") (at 81.28 76.2 0) (unit 2)
+    (in_bom yes) (on_board yes) (dnp no) (fields_autoplaced)
+    (property "Reference" "U1" (at 81.28 66.9757 0)
+      (effects (font (size 1.27 1.27)))
+    )
+    (property "Value" "LM358" (at 81.28 69.3999 0)
+      (effects (font (size 1.27 1.27)))
+    )
+    (property "Footprint" "" (at 81.28 76.2 0)
+      (effects (font (size 1.27 1.27)) hide)
+    )
+    (property "Datasheet" "http://www.ti.com/lit/ds/symlink/lm2904-n.pdf" (at 81.28 76.2 0)
+      (effects (font (size 1.27 1.27)) hide)
+    )
+    (pin "1")
+    (pin "2")
+    (pin "3")
+    (pin "5")
+    (pin "6")
+    (pin "7")
+    (pin "4")
+    (pin "8")
+    (instances
+      (project "sensor"
+        (path "/2513f109-8989-495f-b5d5-45fde763de5f"
+          (reference "U1") (unit 2)
+        )
+      )
