File: Schematic/audio.kicad_sch (KiCad schematic)
At the start: 9 parts, among them J4 Conn_02x01, U1 LM386

Commit message: initial CB design
Parts:
- added C6: .1uF, Capacitor_SMD:C_0805_2012Metric_Pad1.18x1.45mm_HandSolder, symbol Device:C
- added R1: 0, Resistor_SMD:R_1206_3216Metric_Pad1.30x1.75mm_HandSolder, symbol Device:R_US
- C1, C5: footprint (none) -> Capacitor_SMD:C_1206_3216Metric_Pad1.33x1.80mm_HandSolder
- C4: footprint (none) -> Capacitor_THT:CP_Radial_D10.0mm_P5.00mm
- C6: footprint (none) -> Capacitor_THT:CP_Radial_D4.0mm_P2.00mm
- J4: footprint (none) -> Connector_PinHeader_2.54mm:PinHeader_2x01_P2.54mm_Vertical
- R1, R2: footprint (none) -> Resistor_SMD:R_1206_3216Metric_Pad1.30x1.75mm_HandSolder
- U1: footprint (none) -> Package_DIP:DIP-8_W7.62mm
Connections:
- net +12V: now also C6.1
- net Earth renamed GNDA
- net GNDA: now also C6.2, R1.2
- new net GND: R1.1

Commit message: Added stuff from today
Changed lines of the file:
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@@
     )
     (property "Value" "GND" (at 69.2658 76.327 0)
-      (effects (font (size 1.27 1.27)) hide)
+      (effects (font (size 1.27 1.27)))
     )
     (property "Footprint" "" (at 73.66 76.2 0)

Commit message: Added sensors. Fixed other stuff.
Parts:
- J4: footprint Connector_PinHeader_2.54mm:PinHeader_2x01_P2.54mm_Vertical -> Connector_JST:JST_VH_B2P-VH-B_1x02_P3.96mm_Vertical
Changed lines of the file:
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@@
       (effects (font (size 1.27 1.27)) (justify left))
     )
-    (property "Footprint" "Connector_PinHeader_2.54mm:PinHeader_2x01_P2.54mm_Vertical" (at 137.16 66.04 0)
+    (property "Footprint" "Connector_JST:JST_VH_B2P-VH-B_1x02_P3.96mm_Vertical" (at 137.16 66.04 0)
       (effects (font (size 1.27 1.27)) hide)
     )

Commit message: Mostly finallized PCB
Parts:
- J4: value Conn_02x01 -> AUDIO_OUT
Changed lines of the file:
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@@
   (symbol (lib_id "Connector_Generic:Conn_02x01") (at 137.16 66.04 270) (unit 1)
     (in_bom yes) (on_board yes) (dnp no) (fields_autoplaced)
-    (property "Reference" "J4" (at 139.7 66.675 90)
+    (property "Reference" "J4" (at 139.192 66.0979 90)
       (effects (font (size 1.27 1.27)) (justify left))
     )
-    (property "Value" "Conn_02x01" (at 139.7 69.215 90)
+    (property "Value" "AUDIO_OUT" (at 139.192 68.5221 90)
       (effects (font (size 1.27 1.27)) (justify left))
     )

Commit message: Added images
Parts:
- R1: value 20k -> 800
Changed lines of the file:
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@@
       (effects (font (size 1.27 1.27)) (justify right))
     )
-    (property "Value" "20k" (at 88.9 65.405 0)
+    (property "Value" "800" (at 88.9 65.405 0)
       (effects (font (size 1.27 1.27)) (justify right))
     )

Commit message: Added Cap to osilator, and fixed posible issues with signals near it.
Parts:
- C6: footprint Capacitor_SMD:C_0805_2012Metric_Pad1.18x1.45mm_HandSolder -> Capacitor_SMD:C_1206_3216Metric_Pad1.33x1.80mm_HandSolder
Changed lines of the file:
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@@
   (symbol (lib_id "Device:C") (at 95.25 41.91 0) (unit 1)
     (in_bom yes) (on_board yes) (dnp no)
-    (property "Reference" "C6" (at 93.98 48.26 0)
+    (property "Reference" "C6" (at 88.9 41.91 0)
       (effects (font (size 1.27 1.27)) (justify left))
     )
@@
       (effects (font (size 1.27 1.27)) (justify left))
     )
-    (property "Footprint" "Capacitor_SMD:C_0805_2012Metric_Pad1.18x1.45mm_HandSolder" (at 96.2152 45.72 0)
+    (property "Footprint" "Capacitor_SMD:C_1206_3216Metric_Pad1.33x1.80mm_HandSolder" (at 96.2152 45.72 0)
       (effects (font (size 1.27 1.27)) hide)
     )

Commit message: relabeld all of the components so they have more resonable numbers
Parts:
- renumbered J4 to J6
Changed lines of the file:
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@@
       (project "Schematic"
         (path "/ced54cd9-3b34-40e4-aa66-964aaab81b0a/3dc37a54-006b-430f-992a-c37d5e0558dd"
-          (reference "R3") (unit 1)
+          (reference "R41") (unit 1)
         )
       )
@@
       (project "Schematic"
         (path "/ced54cd9-3b34-40e4-aa66-964aaab81b0a/3dc37a54-006b-430f-992a-c37d5e0558dd"
-          (reference "C8") (unit 1)
+          (reference "C11") (unit 1)
         )
       )
@@
         )
         (path "/ced54cd9-3b34-40e4-aa66-964aaab81b0a/3dc37a54-006b-430f-992a-c37d5e0558dd"
-          (reference "#PWR038") (unit 1)
+          (reference "#PWR044") (unit 1)
         )
       )
@@
         )
         (path "/ced54cd9-3b34-40e4-aa66-964aaab81b0a/3dc37a54-006b-430f-992a-c37d5e0558dd"
-          (reference "C11") (unit 1)
+          (reference "C9") (unit 1)
         )
       )
@@
   (symbol (lib_id "Connector_Generic:Conn_02x01") (at 137.16 66.04 270) (unit 1)
     (in_bom yes) (on_board yes) (dnp no) (fields_autoplaced)
-    (property "Reference" "J4" (at 139.192 66.0979 90)
+    (property "Reference" "J6" (at 139.192 66.0979 90)
       (effects (font (size 1.27 1.27)) (justify left))
     )
@@
       (project "Schematic"
         (path "/ced54cd9-3b34-40e4-aa66-964aaab81b0a/3dc37a54-006b-430f-992a-c37d5e0558dd"
-          (reference "J4") (unit 1)
+          (reference "J6") (unit 1)
         )
       )
@@
   (symbol (lib_id "power:GNDA") (at 133.35 78.74 0) (unit 1)
     (in_bom yes) (on_board yes) (dnp no) (fields_autoplaced)
-    (property "Reference" "#PWR039" (at 133.35 85.09 0)
+    (property "Reference" "#PWR046" (at 133.35 85.09 0)
       (effects (font (size 1.27 1.27)) hide)
     )
@@
       (project "Schematic"
         (path "/ced54cd9-3b34-40e4-aa66-964aaab81b0a/3dc37a54-006b-430f-992a-c37d5e0558dd"
-          (reference "#PWR039") (unit 1)
+          (reference "#PWR046") (unit 1)
         )
       )
@@
       (project "Schematic"
         (path "/ced54cd9-3b34-40e4-aa66-964aaab81b0a/3dc37a54-006b-430f-992a-c37d5e0558dd"
-          (reference "C9") (unit 1)
+          (reference "C12") (unit 1)
         )
       )
@@
   (symbol (lib_id "power:GNDA") (at 105.41 44.45 180) (unit 1)
     (in_bom yes) (on_board yes) (dnp no) (fields_autoplaced)
-    (property "Reference" "#PWR030" (at 105.41 38.1 0)
+    (property "Reference" "#PWR045" (at 105.41 38.1 0)
       (effects (font (size 1.27 1.27)) hide)
     )
@@
       (project "Schematic"
         (path "/ced54cd9-3b34-40e4-aa66-964aaab81b0a/3dc37a54-006b-430f-992a-c37d5e0558dd"
-          (reference "#PWR030") (unit 1)
+          (reference "#PWR045") (unit 1)
         )
       )
@@
       (project "Schematic"
         (path "/ced54cd9-3b34-40e4-aa66-964aaab81b0a/3dc37a54-006b-430f-992a-c37d5e0558dd"
-          (reference "R4") (unit 1)
+          (reference "R44") (unit 1)
         )
       )
@@
   (symbol (lib_id "power:+12V") (at 66.04 38.1 0) (unit 1)
     (in_bom yes) (on_board yes) (dnp no) (fields_autoplaced)
-    (property "Reference" "#PWR032" (at 66.04 41.91 0)
+    (property "Reference" "#PWR043" (at 66.04 41.91 0)
       (effects (font (size 1.27 1.27)) hide)
     )
@@
       (project "Schematic"
         (path "/ced54cd9-3b34-40e4-aa66-964aaab81b0a/3dc37a54-006b-430f-992a-c37d5e0558dd"
-          (reference "#PWR032") (unit 1)
+          (reference "#PWR043") (unit 1)
         )
       )
@@
       (project "Schematic"
         (path "/ced54cd9-3b34-40e4-aa66-964aaab81b0a/3dc37a54-006b-430f-992a-c37d5e0558dd"
-          (reference "C10") (unit 1)
+          (reference "C13") (unit 1)
         )
       )
@@
       (project "Schematic"
         (path "/ced54cd9-3b34-40e4-aa66-964aaab81b0a/3dc37a54-006b-430f-992a-c37d5e0558dd"
-          (reference "U3") (unit 1)
+          (reference "U4") (unit 1)
         )
       )
@@
       (project "Schematic"
         (path "/ced54cd9-3b34-40e4-aa66-964aaab81b0a/3dc37a54-006b-430f-992a-c37d5e0558dd"
-          (reference "R7") (unit 1)
+          (reference "R42") (unit 1)
         )
       )
@@
       (project "Schematic"
         (path "/ced54cd9-3b34-40e4-aa66-964aaab81b0a/3dc37a54-006b-430f-992a-c37d5e0558dd"
-          (reference "R5") (unit 1)
+          (reference "R43") (unit 1)
         )
       )
@@
       (project "Schematic"
         (path "/ced54cd9-3b34-40e4-aa66-964aaab81b0a/3dc37a54-006b-430f-992a-c37d5e0558dd"
-          (reference "C7") (unit 1)
-        )
-      )
+          (reference "C10") (unit 1)
+        )
+      )
