File: Schematic/keypad.kicad_sch (KiCad schematic)
At the start: 9 parts, among them J2 Conn_01x08

Commit message: initial CB design
Parts:
- R10, R11, R12, R13, R14, R15, R8, R9: footprint Resistor_SMD:R_0805_2012Metric_Pad1.20x1.40mm_HandSolder -> Resistor_SMD:R_1206_3216Metric_Pad1.30x1.75mm_HandSolder
Connections:
- net PB7: now also R15.1
Changed lines of the file:
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@@
+    (stroke (width 0) (type default))
+  )
+  (wire (pts (xy 40.64 43.18) (xy 41.91 43.18))
+    (stroke (width 0) (type default))
+  )
+  (wire (pts (xy 40.64 49.53) (xy 40.64 43.18))
+    (stroke (width 0) (type default))
+  )
+  (wire (pts (xy 27.94 44.45) (xy 29.21 44.45))
+    (stroke (width 0) (type default))
+  )
+  (wire (pts (xy 27.94 34.29) (xy 29.21 34.29))
+    (stroke (width 0) (type default))
+  )
+  (wire (pts (xy 40.64 30.48) (xy 41.91 30.48))
+    (stroke (width 0) (type default))
+  )
+  (wire (pts (xy 36.83 19.05) (xy 41.91 19.05))
+    (stroke (width 0) (type default))
+  )
+  (wire (pts (xy 38.1 35.56) (xy 38.1 34.29))
+    (stroke (width 0) (type default))
+  )
+  (wire (pts (xy 39.37 29.21) (xy 39.37 33.02))
+    (stroke (width 0) (type default))
+  )
+  (wire (pts (xy 27.94 29.21) (xy 29.21 29.21))
+    (stroke (width 0) (type default))
+  )
+  (wire (pts (xy 27.94 39.37) (xy 29.21 39.37))
+    (stroke (width 0) (type default))
+  )
+  (wire (pts (xy 40.64 24.13) (xy 40.64 30.48))
+    (stroke (width 0) (type default))
+  )
+  (wire (pts (xy 38.1 35.56) (xy 41.91 35.56))
+    (stroke (width 0) (type default))
+  )
+  (wire (pts (xy 38.1 39.37) (xy 38.1 38.1))
+    (stroke (width 0) (type default))
+  )
+  (wire (pts (xy 36.83 54.61) (xy 41.91 54.61))
+    (stroke (width 0) (type default))
+  )
+  (wire (pts (xy 38.1 34.29) (xy 36.83 34.29))
+    (stroke (width 0) (type default))
+  )
+  (wire (pts (xy 27.94 24.13) (xy 29.21 24.13))
+    (stroke (width 0) (type default))
+  )
+  (wire (pts (xy 27.94 19.05) (xy 29.21 19.05))
+    (stroke (width 0) (type default))
+  )
+  (wire (pts (xy 36.83 44.45) (xy 39.37 44.45))
+    (stroke (width 0) (type default))
+  )
+  (wire (pts (xy 41.91 54.61) (xy 41.91 45.72))
+    (stroke (width 0) (type default))
+  )
+  (wire (pts (xy 27.94 49.53) (xy 29.21 49.53))
+    (stroke (width 0) (type default))
+  )
+  (wire (pts (xy 41.91 27.94) (xy 41.91 19.05))
+    (stroke (width 0) (type default))
+  )
+  (wire (pts (xy 36.83 24.13) (xy 40.64 24.13))
+    (stroke (width 0) (type default))
+  )
+  (wire (pts (xy 38.1 38.1) (xy 41.91 38.1))
+    (stroke (width 0) (type default))
+  )
+  (wire (pts (xy 36.83 39.37) (xy 38.1 39.37))
+    (stroke (width 0) (type default))
+  )
+  (wire (pts (xy 36.83 49.53) (xy 40.64 49.53))
+    (stroke (width 0) (type default))
+  )
+  (wire (pts (xy 36.83 29.21) (xy 39.37 29.21))
     (stroke (width 0) (type default))
   )
@@
     (stroke (width 0) (type default))
   )
-  (wire (pts (xy 40.64 43.18) (xy 41.91 43.18))
-    (stroke (width 0) (type default))
-  )
-  (wire (pts (xy 40.64 49.53) (xy 40.64 43.18))
-    (stroke (width 0) (type default))
-  )
-  (wire (pts (xy 27.94 44.45) (xy 29.21 44.45))
-    (stroke (width 0) (type default))
-  )
-  (wire (pts (xy 27.94 34.29) (xy 29.21 34.29))
-    (stroke (width 0) (type default))
-  )
-  (wire (pts (xy 40.64 30.48) (xy 41.91 30.48))
-    (stroke (width 0) (type default))
-  )
-  (wire (pts (xy 36.83 19.05) (xy 41.91 19.05))
-    (stroke (width 0) (type default))
-  )
-  (wire (pts (xy 38.1 35.56) (xy 38.1 34.29))
-    (stroke (width 0) (type default))
-  )
-  (wire (pts (xy 39.37 29.21) (xy 39.37 33.02))
-    (stroke (width 0) (type default))
-  )
-  (wire (pts (xy 27.94 29.21) (xy 29.21 29.21))
-    (stroke (width 0) (type default))
-  )
-  (wire (pts (xy 27.94 39.37) (xy 29.21 39.37))
-    (stroke (width 0) (type default))
-  )
-  (wire (pts (xy 40.64 24.13) (xy 40.64 30.48))
-    (stroke (width 0) (type default))
-  )
-  (wire (pts (xy 38.1 35.56) (xy 41.91 35.56))
-    (stroke (width 0) (type default))
-  )
-  (wire (pts (xy 38.1 39.37) (xy 38.1 38.1))
-    (stroke (width 0) (type default))
-  )
-  (wire (pts (xy 36.83 54.61) (xy 41.91 54.61))
-    (stroke (width 0) (type default))
-  )
-  (wire (pts (xy 38.1 34.29) (xy 36.83 34.29))
-    (stroke (width 0) (type default))
-  )
-  (wire (pts (xy 27.94 24.13) (xy 29.21 24.13))
-    (stroke (width 0) (type default))
-  )
-  (wire (pts (xy 27.94 19.05) (xy 29.21 19.05))
-    (stroke (width 0) (type default))
-  )
-  (wire (pts (xy 36.83 44.45) (xy 39.37 44.45))
-    (stroke (width 0) (type default))
-  )
-  (wire (pts (xy 41.91 54.61) (xy 41.91 45.72))
-    (stroke (width 0) (type default))
-  )
-  (wire (pts (xy 27.94 49.53) (xy 29.21 49.53))
-    (stroke (width 0) (type default))
-  )
-  (wire (pts (xy 41.91 27.94) (xy 41.91 19.05))
-    (stroke (width 0) (type default))
-  )
-  (wire (pts (xy 36.83 24.13) (xy 40.64 24.13))
-    (stroke (width 0) (type default))
-  )
-  (wire (pts (xy 38.1 38.1) (xy 41.91 38.1))
-    (stroke (width 0) (type default))
-  )
-  (wire (pts (xy 36.83 39.37) (xy 38.1 39.37))
-    (stroke (width 0) (type default))
-  )
-  (wire (pts (xy 36.83 49.53) (xy 40.64 49.53))
-    (stroke (width 0) (type default))
-  )
-  (wire (pts (xy 36.83 29.21) (xy 39.37 29.21))
-    (stroke (width 0) (type default))
-  )
   (wire (pts (xy 39.37 33.02) (xy 41.91 33.02))
     (stroke (width 0) (type default))
@@
     (stroke (width 0) (type default))
   )
-  (global_label "PB7" (shape input) (at 27.94 54.6504 180) (fields_autoplaced)
-    (effects (font (size 1.27 1.27)) (justify right))
-    (property "Intersheetrefs" "${INTERSHEET_REFS}" (at 21.2847 54.6504 0)
+  (global_label "PB7" (shape input) (at 27.94 54.61 180) (fields_autoplaced)
+    (effects (font (size 1.27 1.27)) (justify right))
+    (property "Intersheetrefs" "${INTERSHEET_REFS}" (at 21.2847 54.61 0)
       (effects (font (size 1.27 1.27)) (justify right) hide)
     )
@@
       (effects (font (size 1.27 1.27)))
     )
-    (property "Footprint" "Resistor_SMD:R_0805_2012Metric_Pad1.20x1.40mm_HandSolder" (at 33.02 41.148 90)
+    (property "Footprint" "Resistor_SMD:R_1206_3216Metric_Pad1.30x1.75mm_HandSolder" (at 33.02 41.148 90)
       (effects (font (size 1.27 1.27)) hide)
     )
@@
       (effects (font (size 1.27 1.27)))
     )
-    (property "Footprint" "Resistor_SMD:R_0805_2012Metric_Pad1.20x1.40mm_HandSolder" (at 33.02 51.308 90)
+    (property "Footprint" "Resistor_SMD:R_1206_3216Metric_Pad1.30x1.75mm_HandSolder" (at 33.02 51.308 90)
       (effects (font (size 1.27 1.27)) hide)
     )
@@
       (effects (font (size 1.27 1.27)))
     )
-    (property "Footprint" "Resistor_SMD:R_0805_2012Metric_Pad1.20x1.40mm_HandSolder" (at 33.02 25.908 90)
+    (property "Footprint" "Resistor_SMD:R_1206_3216Metric_Pad1.30x1.75mm_HandSolder" (at 33.02 25.908 90)
       (effects (font (size 1.27 1.27)) hide)
     )
@@
       (effects (font (size 1.27 1.27)))
     )
-    (property "Footprint" "Resistor_SMD:R_0805_2012Metric_Pad1.20x1.40mm_HandSolder" (at 33.02 20.828 90)
+    (property "Footprint" "Resistor_SMD:R_1206_3216Metric_Pad1.30x1.75mm_HandSolder" (at 33.02 20.828 90)
       (effects (font (size 1.27 1.27)) hide)
     )
@@
       (effects (font (size 1.27 1.27)))
     )
-    (property "Footprint" "Resistor_SMD:R_0805_2012Metric_Pad1.20x1.40mm_HandSolder" (at 33.02 36.068 90)
+    (property "Footprint" "Resistor_SMD:R_1206_3216Metric_Pad1.30x1.75mm_HandSolder" (at 33.02 36.068 90)
       (effects (font (size 1.27 1.27)) hide)
     )
@@
       (effects (font (size 1.27 1.27)))
     )
-    (property "Footprint" "Resistor_SMD:R_0805_2012Metric_Pad1.20x1.40mm_HandSolder" (at 33.02 30.988 90)
+    (property "Footprint" "Resistor_SMD:R_1206_3216Metric_Pad1.30x1.75mm_HandSolder" (at 33.02 30.988 90)
       (effects (font (size 1.27 1.27)) hide)
     )
@@
       (effects (font (size 1.27 1.27)))
     )
-    (property "Footprint" "Resistor_SMD:R_0805_2012Metric_Pad1.20x1.40mm_HandSolder" (at 33.02 46.228 90)
+    (property "Footprint" "Resistor_SMD:R_1206_3216Metric_Pad1.30x1.75mm_HandSolder" (at 33.02 46.228 90)
       (effects (font (size 1.27 1.27)) hide)
     )
@@
       (effects (font (size 1.27 1.27)))
     )
-    (property "Footprint" "Resistor_SMD:R_0805_2012Metric_Pad1.20x1.40mm_HandSolder" (at 33.02 56.388 90)
-      (effects (font (size 1.27 1.27)) hide)
-    )
+    (property "Footprint" "Resistor_SMD:R_1206_3216Metric_Pad1.30x1.75mm_HandSolder" (at 33.02 56.388 90)
+      (effects (font (size 1.27 1.27)) hide)
+    )

Commit message: Mostly finallized PCB
Parts:
- J2: value Conn_01x08 -> KEYPAD
Changed lines of the file:
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@@
   (symbol (lib_id "Connector_Generic:Conn_01x08") (at 46.99 35.56 0) (unit 1)
     (in_bom yes) (on_board yes) (dnp no) (fields_autoplaced)
-    (property "Reference" "J2" (at 49.53 36.195 0)
+    (property "Reference" "J2" (at 49.022 35.6179 0)
       (effects (font (size 1.27 1.27)) (justify left))
     )
-    (property "Value" "Conn_01x08" (at 49.53 38.735 0)
+    (property "Value" "KEYPAD" (at 49.022 38.0421 0)
       (effects (font (size 1.27 1.27)) (justify left))
     )

Commit message: Lab fixes
Parts:
- added R6, R61, R62, R63: 10k, Resistor_SMD:R_1206_3216Metric_Pad1.30x1.75mm_HandSolder, symbol Device:R
Connections:
- net at J2.5 (Pin_5), R12.2: now also R63.2
- net at J2.7 (Pin_7), R14.2: now also R61.2
- net at J2.6 (Pin_6), R13.2: now also R62.2
- net at J2.8 (Pin_8), R15.2: now also R6.2
- new net GND: R6.1, R61.1, R62.1, R63.1
Other:
- moved on the sheet: R12, R13, R14, R15

Commit message: relabeld all of the components so they have more resonable numbers
Parts:
- renumbered J2 to J5, R12 to R29, R63 to R30, R13 to R31, R62 to R32, R14 to R33, R15 to R34, R8 to R35, R9 to R36, R10 to R37, R11 to R38, R61 to R39, R6 to R40
Changed lines of the file:
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@@
   (symbol (lib_id "Device:R") (at 26.67 39.37 90) (unit 1)
     (in_bom yes) (on_board yes) (dnp no)
-    (property "Reference" "R12" (at 26.67 36.83 90)
+    (property "Reference" "R29" (at 26.67 36.83 90)
       (effects (font (size 1.27 1.27)))
     )
@@
       (project "Schematic"
         (path "/ced54cd9-3b34-40e4-aa66-964aaab81b0a/b3c6fc2a-9568-48a3-9317-55c435503364"
-          (reference "R12") (unit 1)
+          (reference "R29") (unit 1)
         )
       )
@@
   (symbol (lib_id "Device:R") (at 26.67 55.88 90) (unit 1)
     (in_bom yes) (on_board yes) (dnp no)
-    (property "Reference" "R62" (at 26.67 53.34 90)
+    (property "Reference" "R32" (at 26.67 53.34 90)
       (effects (font (size 1.27 1.27)))
     )
@@
       (project "Schematic"
         (path "/ced54cd9-3b34-40e4-aa66-964aaab81b0a/b3c6fc2a-9568-48a3-9317-55c435503364"
-          (reference "R62") (unit 1)
+          (reference "R32") (unit 1)
         )
       )
@@
   (symbol (lib_id "Device:R") (at 34.29 64.77 90) (unit 1)
     (in_bom yes) (on_board yes) (dnp no)
-    (property "Reference" "R61" (at 34.29 62.23 90)
+    (property "Reference" "R39" (at 34.29 62.23 90)
       (effects (font (size 1.27 1.27)))
     )
@@
       (project "Schematic"
         (path "/ced54cd9-3b34-40e4-aa66-964aaab81b0a/b3c6fc2a-9568-48a3-9317-55c435503364"
-          (reference "R61") (unit 1)
+          (reference "R39") (unit 1)
         )
       )
@@
   (symbol (lib_id "Device:R") (at 36.83 73.66 90) (unit 1)
     (in_bom yes) (on_board yes) (dnp no)
-    (property "Reference" "R6" (at 36.83 71.12 90)
+    (property "Reference" "R40" (at 36.83 71.12 90)
       (effects (font (size 1.27 1.27)))
     )
@@
       (project "Schematic"
         (path "/ced54cd9-3b34-40e4-aa66-964aaab81b0a/b3c6fc2a-9568-48a3-9317-55c435503364"
-          (reference "R6") (unit 1)
+          (reference "R40") (unit 1)
         )
       )
@@
   (symbol (lib_id "Device:R") (at 26.67 60.96 90) (unit 1)
     (in_bom yes) (on_board yes) (dnp no)
-    (property "Reference" "R14" (at 26.67 58.42 90)
+    (property "Reference" "R33" (at 26.67 58.42 90)
       (effects (font (size 1.27 1.27)))
     )
@@
       (project "Schematic"
         (path "/ced54cd9-3b34-40e4-aa66-964aaab81b0a/b3c6fc2a-9568-48a3-9317-55c435503364"
-          (reference "R14") (unit 1)
+          (reference "R33") (unit 1)
         )
       )
@@
         )
         (path "/ced54cd9-3b34-40e4-aa66-964aaab81b0a/b3c6fc2a-9568-48a3-9317-55c435503364"
-          (reference "#PWR078") (unit 1)
+          (reference "#PWR042") (unit 1)
         )
       )
@@
         )
         (path "/ced54cd9-3b34-40e4-aa66-964aaab81b0a/b3c6fc2a-9568-48a3-9317-55c435503364"
-          (reference "#PWR079") (unit 1)
+          (reference "#PWR041") (unit 1)
         )
       )
@@
   (symbol (lib_id "Device:R") (at 33.02 24.13 90) (unit 1)
     (in_bom yes) (on_board yes) (dnp no)
-    (property "Reference" "R9" (at 33.02 21.59 90)
+    (property "Reference" "R36" (at 33.02 21.59 90)
       (effects (font (size 1.27 1.27)))
     )
@@
       (project "Schematic"
         (path "/ced54cd9-3b34-40e4-aa66-964aaab81b0a/b3c6fc2a-9568-48a3-9317-55c435503364"
-          (reference "R9") (unit 1)
+          (reference "R36") (unit 1)
         )
       )
@@
   (symbol (lib_id "Connector_Generic:Conn_01x08") (at 46.99 35.56 0) (unit 1)
     (in_bom yes) (on_board yes) (dnp no) (fields_autoplaced)
-    (property "Reference" "J2" (at 49.022 35.6179 0)
+    (property "Reference" "J5" (at 49.022 35.6179 0)
       (effects (font (size 1.27 1.27)) (justify left))
     )
@@
       (project "Schematic"
         (path "/ced54cd9-3b34-40e4-aa66-964aaab81b0a/b3c6fc2a-9568-48a3-9317-55c435503364"
-          (reference "J2") (unit 1)
+          (reference "J5") (unit 1)
         )
       )
@@
   (symbol (lib_id "Device:R") (at 33.02 19.05 90) (unit 1)
     (in_bom yes) (on_board yes) (dnp no)
-    (property "Reference" "R8" (at 33.02 16.51 90)
+    (property "Reference" "R35" (at 33.02 16.51 90)
       (effects (font (size 1.27 1.27)))
     )
@@
       (project "Schematic"
         (path "/ced54cd9-3b34-40e4-aa66-964aaab81b0a/b3c6fc2a-9568-48a3-9317-55c435503364"
-          (reference "R8") (unit 1)
+          (reference "R35") (unit 1)
         )
       )
@@
         )
         (path "/ced54cd9-3b34-40e4-aa66-964aaab81b0a/b3c6fc2a-9568-48a3-9317-55c435503364"
-          (reference "#PWR081") (unit 1)
+          (reference "#PWR039") (unit 1)
         )
       )
@@
   (symbol (lib_id "Device:R") (at 33.02 34.29 90) (unit 1)
     (in_bom yes) (on_board yes) (dnp no)
-    (property "Reference" "R11" (at 33.02 31.75 90)
+    (property "Reference" "R38" (at 33.02 31.75 90)
       (effects (font (size 1.27 1.27)))
     )
@@
       (project "Schematic"
         (path "/ced54cd9-3b34-40e4-aa66-964aaab81b0a/b3c6fc2a-9568-48a3-9317-55c435503364"
-          (reference "R11") (unit 1)
+          (reference "R38") (unit 1)
         )
       )
@@
         )
         (path "/ced54cd9-3b34-40e4-aa66-964aaab81b0a/b3c6fc2a-9568-48a3-9317-55c435503364"
-          (reference "#PWR080") (unit 1)
+          (reference "#PWR040") (unit 1)
         )
       )
@@
   (symbol (lib_id "Device:R") (at 26.67 44.45 90) (unit 1)
     (in_bom yes) (on_board yes) (dnp no)
-    (property "Reference" "R63" (at 26.67 41.91 90)
+    (property "Reference" "R30" (at 26.67 41.91 90)
       (effects (font (size 1.27 1.27)))
     )
@@
       (project "Schematic"
         (path "/ced54cd9-3b34-40e4-aa66-964aaab81b0a/b3c6fc2a-9568-48a3-9317-55c435503364"
-          (reference "R63") (unit 1)
+          (reference "R30") (unit 1)
         )
       )
@@
   (symbol (lib_id "Device:R") (at 33.02 29.21 90) (unit 1)
     (in_bom yes) (on_board yes) (dnp no)
-    (property "Reference" "R10" (at 33.02 26.67 90)
+    (property "Reference" "R37" (at 33.02 26.67 90)
       (effects (font (size 1.27 1.27)))
     )
@@
       (project "Schematic"
         (path "/ced54cd9-3b34-40e4-aa66-964aaab81b0a/b3c6fc2a-9568-48a3-9317-55c435503364"
-          (reference "R10") (unit 1)
+          (reference "R37") (unit 1)
         )
       )
@@
   (symbol (lib_id "Device:R") (at 26.67 50.8 90) (unit 1)
     (in_bom yes) (on_board yes) (dnp no)
-    (property "Reference" "R13" (at 26.67 48.26 90)
+    (property "Reference" "R31" (at 26.67 48.26 90)
       (effects (font (size 1.27 1.27)))
     )
@@
       (project "Schematic"
         (path "/ced54cd9-3b34-40e4-aa66-964aaab81b0a/b3c6fc2a-9568-48a3-9317-55c435503364"
-          (reference "R13") (unit 1)
+          (reference "R31") (unit 1)
         )
       )
@@
   (symbol (lib_id "Device:R") (at 26.67 69.85 90) (unit 1)
     (in_bom yes) (on_board yes) (dnp no)
-    (property "Reference" "R15" (at 25.4 67.31 90)
+    (property "Reference" "R34" (at 25.4 67.31 90)
       (effects (font (size 1.27 1.27)))
     )
@@
       (project "Schematic"
         (path "/ced54cd9-3b34-40e4-aa66-964aaab81b0a/b3c6fc2a-9568-48a3-9317-55c435503364"
-          (reference "R15") (unit 1)
-        )
-      )
+          (reference "R34") (unit 1)
+        )
+      )
